Commit message: Add kingfisher_localization: the SBG following VRX topics
The boat now publishes what the sim does:
ros2 launch kingfisher_localization localization.launch.py

- sensors/imu/imu/data and sensors/gps/gps/fix, VRX's names, in
  kingfisher/imu_link (ENU orientation, FLU rates) and kingfisher/gps_link;
- odom and odom -> kingfisher/base_link: ENU about the site datum, the
  same origin as the Gazebo world (not UTM, ~2 deg off at the lake),
  twist in base_link;
- map -> odom, the identity (the RTK INS doesn't drift), and
  map -> <point> for the site points (config/sites/lac_symphonie.yaml).

sbg_localization converts the driver's raw sbg/* (NED) messages and
replaces localization_manager for Kingfisher. Without a valid position
(indoors), odom is still published, held at the last position (the
datum if none) with a large variance. The driver config moves here
from the driver checkout, which is back to upstream.

kingfisher_description: imu_link_ned (roll pi under imu_link), the
frame of the raw sbg/* messages.

Co-Authored-By: Claude Opus 5.5 <noreply@anthropic.com>

File: kingfisher_description/urdf/kingfisher.urdf.xacro (robot description, xacro)
@@ -16,4 +16,11 @@
   <xacro:kingfisher_thruster prefix="right" position="-0.53 -0.3776 -0.16"/>
   <xacro:kingfisher_frame name="imu" xyz="-0.15 0 0.14"/>
+  <!-- FRD: the frame of the SBG driver's raw sbg/* messages (NED convention) -->
+  <link name="imu_link_ned"/>
+  <joint name="imu_ned_joint" type="fixed">
+    <origin xyz="0 0 0" rpy="${pi} 0 0"/>
+    <parent link="imu_link"/>
+    <child link="imu_link_ned"/>
+  </joint>
   <!-- The SBG NavSatFix is really at the primary antenna -->
   <xacro:kingfisher_frame name="gps" parent="imu_link"/>
